File: RP2040_SMPS/RP2040_SMPS.kicad_sch (KiCad schematic)
At the start: 81 parts, among them J1 debug, J2 Conn_01x02, J3 USB_B_Mini, J4 Conn_01x01, J5 Screw_Terminal_01x02, J6 Screw_Terminal_01x02, J7 Conn_01x01, Q1 Q_NMOS_DGS, Q2 Q_NMOS_DGS, Q3 Q_NMOS_DGS, Q4 Q_NMOS_DGS, Q5 Q_NMOS_DGS, SW1 SW_SPST, SW2 SW_SPST, SW3 SW_SPST, SW4 SW_SPST, U1 LM4040DBZ-3.0, U2 W25Q128JVS, U3 RP2040, U4 D1213A-02SM, U5 Opamp_Dual, Y1 ABLS-12.000MHZ-B4-T

Commit message: Update RP2040_SMPS.kicad_sch
Connections:
- net at L2.2, Q4.1 (D): now also Q2.3 (S); no longer Q2.1 (D)
- net at C16.1, R12.2, R15.2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: now also Q1.1 (D); no longer Q1.3 (S)
- net at L2.1, Q3.1 (D): now also Q1.3 (S); no longer Q1.1 (D)
- net at C17.1, L1.1: now also Q2.1 (D); no longer Q2.3 (S)
Other:
- moved on the sheet: H1, H2, H3, H4, Q2, R8
Changed lines of the file:
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@@
   (junction (at 246.38 237.49) (diameter 0) (color 0 0 0 0)
   )
+  (junction (at 30.48 153.67) (diameter 0) (color 0 0 0 0)
+  )
   (junction (at 240.03 212.09) (diameter 0) (color 0 0 0 0)
   )
@@
     (stroke (width 0) (type default) (color 0 0 0 0))
   )
-  (wire (pts (xy 38.1 139.7) (xy 38.1 142.24))
+  (wire (pts (xy 30.48 139.7) (xy 30.48 142.24))
     (stroke (width 0) (type default) (color 0 0 0 0))
   )
@@
     (stroke (width 0) (type default) (color 0 0 0 0))
   )
-  (wire (pts (xy 38.1 149.86) (xy 38.1 153.67))
+  (wire (pts (xy 30.48 149.86) (xy 30.48 153.67))
     (stroke (width 0) (type default) (color 0 0 0 0))
   )
@@
     (stroke (width 0) (type default) (color 0 0 0 0))
   )
-  (text "reset buton" (at 40.64 151.13 0)
+  (text "reset buton" (at 33.02 151.13 0)
     (effects (font (size 1.27 1.27)) (justify left bottom))
   )
@@
     (effects (font (size 1.27 1.27)) (justify left bottom))
   )
-  (text "Make sure R3 and R4 are close to RP2040" (at 164.465 69.215 0)
+  (text "Make sure R3 and R4 are close to RP2040" (at 165.1 71.12 0)
     (effects (font (size 1.27 1.27)) (justify left bottom))
   )
@@
     (pin "2")
   )
-  (symbol (lib_id "Mechanical:MountingHole") (at 254 114.3 0) (unit 1)
+  (symbol (lib_id "Mechanical:MountingHole") (at 254 116.84 0) (unit 1)
     (in_bom no) (on_board yes)
-    (property "Reference" "H3" (id 0) (at 252.73 110.49 0)
+    (property "Reference" "H3" (id 0) (at 252.73 113.03 0)
       (effects (font (size 1.27 1.27)) (justify left))
     )
-    (property "Value" "MountingHole" (id 1) (at 247.65 119.38 0)
+    (property "Value" "MountingHole" (id 1) (at 247.65 110.49 0)
       (effects (font (size 1.27 1.27)) (justify left))
     )
-    (property "Footprint" "MountingHole:MountingHole_3.2mm_M3" (id 2) (at 254 114.3 0)
+    (property "Footprint" "MountingHole:MountingHole_3.2mm_M3" (id 2) (at 254 116.84 0)
       (effects (font (size 1.27 1.27)) hide)
     )
-    (property "Datasheet" "~" (id 3) (at 254 114.3 0)
+    (property "Datasheet" "~" (id 3) (at 254 116.84 0)
       (effects (font (size 1.27 1.27)) hide)
     )
@@
     (pin "2")
   )
-  (symbol (lib_id "Device:Q_NMOS_DGS") (at 123.19 229.87 0) (mirror x) (unit 1)
+  (symbol (lib_id "Device:Q_NMOS_DGS") (at 123.19 229.87 0) (unit 1)
     (in_bom yes) (on_board yes) (fields_autoplaced)
     (property "Reference" "Q1" (id 0) (at 129.54 228.5999 0)
@@
       (effects (font (size 1.27 1.27)) (justify left))
     )
-    (property "Footprint" "" (id 2) (at 128.27 232.41 0)
+    (property "Footprint" "" (id 2) (at 128.27 227.33 0)
       (effects (font (size 1.27 1.27)) hide)
     )
@@
     (pin "2")
   )
-  (symbol (lib_id "Device:R") (at 38.1 146.05 0) (mirror x) (unit 1)
+  (symbol (lib_id "Device:R") (at 30.48 146.05 0) (mirror x) (unit 1)
     (in_bom yes) (on_board yes)
-    (property "Reference" "R8" (id 0) (at 34.29 144.78 0))
-    (property "Value" "10k" (id 1) (at 34.29 147.32 0))
-    (property "Footprint" "Resistor_SMD:R_0603_1608Metric_Pad0.98x0.95mm_HandSolder" (id 2) (at 36.322 146.05 90)
+    (property "Reference" "R8" (id 0) (at 26.67 144.78 0))
+    (property "Value" "10k" (id 1) (at 26.67 147.32 0))
+    (property "Footprint" "Resistor_SMD:R_0603_1608Metric_Pad0.98x0.95mm_HandSolder" (id 2) (at 28.702 146.05 90)
       (effects (font (size 1.27 1.27)) hide)
     )
-    (property "Datasheet" "~" (id 3) (at 38.1 146.05 0)
+    (property "Datasheet" "~" (id 3) (at 30.48 146.05 0)
       (effects (font (size 1.27 1.27)) hide)
     )
@@
     (pin "2")
   )
-  (symbol (lib_id "Mechanical:MountingHole") (at 254 102.87 0) (unit 1)
+  (symbol (lib_id "Mechanical:MountingHole") (at 254 105.41 0) (unit 1)
     (in_bom no) (on_board yes)
-    (property "Reference" "H1" (id 0) (at 252.73 99.06 0)
+    (property "Reference" "H1" (id 0) (at 252.73 101.6 0)
       (effects (font (size 1.27 1.27)) (justify left))
     )
-    (property "Value" "MountingHole" (id 1) (at 247.65 107.95 0)
+    (property "Value" "MountingHole" (id 1) (at 247.65 99.06 0)
       (effects (font (size 1.27 1.27)) (justify left))
     )
-    (property "Footprint" "MountingHole:MountingHole_3.2mm_M3" (id 2) (at 254 102.87 0)
+    (property "Footprint" "MountingHole:MountingHole_3.2mm_M3" (id 2) (at 254 105.41 0)
       (effects (font (size 1.27 1.27)) hide)
     )
-    (property "Datasheet" "~" (id 3) (at 254 102.87 0)
+    (property "Datasheet" "~" (id 3) (at 254 105.41 0)
       (effects (font (size 1.27 1.27)) hide)
     )
   )
-  (symbol (lib_id "Mechanical:MountingHole") (at 267.97 114.3 0) (unit 1)
+  (symbol (lib_id "Mechanical:MountingHole") (at 270.51 116.84 0) (unit 1)
     (in_bom no) (on_board yes)
-    (property "Reference" "H4" (id 0) (at 266.7 110.49 0)
+    (property "Reference" "H4" (id 0) (at 269.24 113.03 0)
       (effects (font (size 1.27 1.27)) (justify left))
     )
-    (property "Value" "MountingHole" (id 1) (at 261.62 119.38 0)
+    (property "Value" "MountingHole" (id 1) (at 264.16 110.49 0)
       (effects (font (size 1.27 1.27)) (justify left))
     )
-    (property "Footprint" "MountingHole:MountingHole_3.2mm_M3" (id 2) (at 267.97 114.3 0)
+    (property "Footprint" "MountingHole:MountingHole_3.2mm_M3" (id 2) (at 270.51 116.84 0)
       (effects (font (size 1.27 1.27)) hide)
     )
-    (property "Datasheet" "~" (id 3) (at 267.97 114.3 0)
+    (property "Datasheet" "~" (id 3) (at 270.51 116.84 0)
       (effects (font (size 1.27 1.27)) hide)
     )
@@
     (pin "1")
   )
-  (symbol (lib_id "Mechanical:MountingHole") (at 267.97 102.87 0) (unit 1)
+  (symbol (lib_id "Mechanical:MountingHole") (at 270.51 105.41 0) (unit 1)
     (in_bom no) (on_board yes)
-    (property "Reference" "H2" (id 0) (at 266.7 99.06 0)
+    (property "Reference" "H2" (id 0) (at 269.24 101.6 0)
       (effects (font (size 1.27 1.27)) (justify left))
     )
-    (property "Value" "MountingHole" (id 1) (at 261.62 107.95 0)
+    (property "Value" "MountingHole" (id 1) (at 264.16 99.06 0)
       (effects (font (size 1.27 1.27)) (justify left))
     )
-    (property "Footprint" "MountingHole:MountingHole_3.2mm_M3" (id 2) (at 267.97 102.87 0)
+    (property "Footprint" "MountingHole:MountingHole_3.2mm_M3" (id 2) (at 270.51 105.41 0)
       (effects (font (size 1.27 1.27)) hide)
     )
-    (property "Datasheet" "~" (id 3) (at 267.97 102.87 0)
+    (property "Datasheet" "~" (id 3) (at 270.51 105.41 0)
       (effects (font (size 1.27 1.27)) hide)
     )
@@
     (pin "1")
   )
-  (symbol (lib_id "power:+3V3") (at 38.1 139.7 0) (unit 1)
+  (symbol (lib_id "power:+3V3") (at 30.48 139.7 0) (unit 1)
     (in_bom yes) (on_board yes)
-    (property "Reference" "#PWR018" (id 0) (at 38.1 143.51 0)
+    (property "Reference" "#PWR018" (id 0) (at 30.48 143.51 0)
       (effects (font (size 1.27 1.27)) hide)
     )
-    (property "Value" "+3V3" (id 1) (at 38.1 135.89 0))
-    (property "Footprint" "" (id 2) (at 38.1 139.7 0)
+    (property "Value" "+3V3" (id 1) (at 30.48 135.89 0))
+    (property "Footprint" "" (id 2) (at 30.48 139.7 0)
       (effects (font (size 1.27 1.27)) hide)
     )
-    (property "Datasheet" "" (id 3) (at 38.1 139.7 0)
+    (property "Datasheet" "" (id 3) (at 30.48 139.7 0)
       (effects (font (size 1.27 1.27)) hide)
     )
     (pin "1")
   )
-  (symbol (lib_id "Device:Q_NMOS_DGS") (at 177.8 229.87 180) (unit 1)
+  (symbol (lib_id "Device:Q_NMOS_DGS") (at 177.8 229.87 0) (mirror y) (unit 1)
     (in_bom yes) (on_board yes) (fields_autoplaced)
     (property "Reference" "Q2" (id 0) (at 171.45 228.5999 0)
@@
       (effects (font (size 1.27 1.27)) (justify left))
     )
-    (property "Footprint" "" (id 2) (at 172.72 232.41 0)
+    (property "Footprint" "" (id 2) (at 172.72 227.33 0)
       (effects (font (size 1.27 1.27)) hide)
     )
@@
   (symbol (lib_id "Connector_Generic:Conn_01x01") (at 278.13 167.64 180) (unit 1)
     (in_bom no) (on_board yes)
-    (property "Reference" "J4" (id 0) (at 273.05 169.545 0))
+    (property "Reference" "J4" (id 0) (at 274.32 167.64 0))
     (property "Value" "Conn_01x01" (id 1) (at 273.05 172.085 0)
       (effects (font (size 1.27 1.27)) hide)

Commit message: Update RP2040_SMPS.kicad_sch
Parts:
- removed SW1: SW_SPST, SamacSys_Parts:PTS526SK15SMTR2LFS, symbol Switch:SW_SPST
- removed SW3, SW4: SW_SPST, symbol Switch:SW_SPST
- added C21, C22, C27, C28: z, Capacitor_SMD:C_0805_2012Metric_Pad1.18x1.45mm_HandSolder, symbol Device:C
- added C23, C24, C25, C26: 100n, Capacitor_SMD:C_0805_2012Metric_Pad1.18x1.45mm_HandSolder, symbol Device:C
- added J8: Screw_Terminal_01x02, symbol Connector:Screw_Terminal_01x02
- added Q6, Q7: Q_PMOS_DGS, symbol Device:Q_PMOS_DGS
- added R27, R32, R33: 100k, Resistor_SMD:R_0603_1608Metric_Pad0.98x0.95mm_HandSolder, symbol Device:R
- added R28, R29, R30, R31: 10k, Resistor_SMD:R_0603_1608Metric_Pad0.98x0.95mm_HandSolder, symbol Device:R
- added R34, R35, R36, R37: 1k, Resistor_SMD:R_0603_1608Metric_Pad0.98x0.95mm_HandSolder, symbol Device:R
- added SW1: SW_DIP_x08, Button_Switch_THT:SW_DIP_SPSTx08_Slide_9.78x22.5mm_W7.62mm_P2.54mm, symbol Switch:SW_DIP_x08
- added U6, U7, U8: Opamp_Dual, symbol Device:Opamp_Dual
Connections:
- net +3V3: now also SW1.14, SW1.15, SW1.16
- net GND: now also Q3.3 (S), Q4.3 (S), C21.2, C22.2, C23.2, C24.2, C25.2, C26.2, C27.2, C28.2, J8.1 (Pin_1), R31.1, R33.2, SW1.8; no longer R22.1
- net GPIO0: now also R20.2, SW1.2; no longer R19.2
- net GPIO1: now also R19.2, SW1.1; no longer R20.2
- net ~{USB_BOOT}: now also SW1.9
- net +12V: now reaches J6.2 (Pin_2), R12.1, R21.1
- net +12V: now also R22.2, R29.1
- new net: C24.1, R35.1, U6.5 (+)
- new net: C26.1, R37.1, U7.5 (+)
- new net: R28.2, U6.1
- new net: C23.1, R34.1, U6.2 (-)
- new net: R27.1, R31.2, U6.3 (+)
- new net: R29.2, R33.1, U8.3 (+)
- new net: C25.1, R36.1, U7.3 (+)
- new net: R32.1, U7.2 (-), U8.1
- new net: R30.1, R32.2, U8.2 (-)
- new net: R36.2, U7.6 (-), U7.7
- new net: R34.2, U6.6 (-), U6.7
- new net: C21.1, C22.1, J8.2 (Pin_2), Q6.1 (D), R27.2
- new net: Q6.2 (G), Q7.1 (D), R28.1
- new net: C27.1, C28.1, Q6.3 (S), Q7.3 (S), R22.1, R30.2
- new net: Q7.2 (G), U7.1
- new net ref_pwm2: R35.2
- new net ref_pwm3: R37.2
Other:
- moved on the sheet: R19, R20, R22

Commit message: Update RP2040_SMPS.kicad_sch
Other:
- note added: "with 12V in 2A out: inductor/FET current 1v D= 8.8% Imax=22.5A 48A 3.3v Imax=7.27A 14.5A 5V Imax=4.8A 9.6A 48V D=76% Imax=0.5A 4.3A 120V Imax=0.2A 4.3A"
Changed lines of the file:
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@@
+    (effects (font (size 1.27 1.27)) (justify left bottom))
+  )
+  (text "with 12V in 2A\nout:                        inductor/FET current\n1v D= 8.8%  Imax=22.5A             48A\n3.3v        Imax=7.27A             14.5A\n5V          Imax=4.8A              9.6A                                              \n48V D=76%   Imax=0.5A              4.3A   \n120V        Imax=0.2A              4.3A                                             "
+    (at -52.07 228.6 0)
     (effects (font (size 1.27 1.27)) (justify left bottom))
   )
