File: RP2040_SMPS/RP2040_SMPS.kicad_sch (KiCad schematic)
At the start: 104 parts, among them J1 debug, J2 Conn_01x02, J3 USB_B_Mini, J4 Conn_01x01, J5 Screw_Terminal_01x02, J6 Screw_Terminal_01x02, J7 Conn_01x01, J8 Screw_Terminal_01x02, Q1 Q_NMOS_DGS, Q2 Q_NMOS_DGS, Q3 Q_NMOS_DGS, Q4 Q_NMOS_DGS, Q5 Q_NMOS_DGS, Q6 Q_PMOS_DGS, Q7 Q_PMOS_DGS, SW1 SW_DIP_x08, SW2 SW_SPST, U1 LM4040DBZ-3.0, U2 W25Q128JVS, U3 RP2040, U4 D1213A-02SM, U5 Opamp_Dual, U6 Opamp_Dual, U7 Opamp_Dual, U8 Opamp_Dual, Y1 ABLS-12.000MHZ-B4-T

Commit message: j
Parts:
- removed C16: y, Capacitor_SMD:C_0805_2012Metric_Pad1.18x1.45mm_HandSolder, symbol Device:C
- removed C17: x, Capacitor_SMD:C_0805_2012Metric_Pad1.18x1.45mm_HandSolder, symbol Device:C
- removed C18, C21, C22, C27, C28: z, Capacitor_SMD:C_0805_2012Metric_Pad1.18x1.45mm_HandSolder, symbol Device:C
- removed C19, C20, C23, C24, C25, C26: 100n, Capacitor_SMD:C_0805_2012Metric_Pad1.18x1.45mm_HandSolder, symbol Device:C
- removed C4: 22u, Capacitor_SMD:C_0805_2012Metric_Pad1.18x1.45mm_HandSolder, symbol Device:C
- removed D2, D3: 3v, symbol Device:D_Zener_Small
- removed J4, J7: Conn_01x01, Connector_PinSocket_2.54mm:PinSocket_1x01_P2.54mm_Vertical, symbol Connector_Generic:Conn_01x01
- removed J5, J6, J8: Screw_Terminal_01x02, symbol Connector:Screw_Terminal_01x02
- removed L1: L_Small, symbol Device:L_Small
- removed L2: INDUCTOR, symbol pspice:INDUCTOR
- removed Q1, Q2, Q3, Q4, Q5: Q_NMOS_DGS, symbol Device:Q_NMOS_DGS
- removed Q6, Q7: Q_PMOS_DGS, symbol Device:Q_PMOS_DGS
- removed R11, R12, R22: SHUNT, symbol Device:R_Small
- removed R23: e, Resistor_SMD:R_0603_1608Metric_Pad0.98x0.95mm_HandSolder, symbol Device:R
- removed R24, R28, R29, R30, R31: 10k, Resistor_SMD:R_0603_1608Metric_Pad0.98x0.95mm_HandSolder, symbol Device:R
- removed R25, R26, R34, R35, R36, R37: 1k, Resistor_SMD:R_0603_1608Metric_Pad0.98x0.95mm_HandSolder, symbol Device:R
- removed R27, R32, R33: 100k, Resistor_SMD:R_0603_1608Metric_Pad0.98x0.95mm_HandSolder, symbol Device:R
- removed R5, R6: 27, Resistor_SMD:R_0603_1608Metric_Pad0.98x0.95mm_HandSolder, symbol Device:R
- removed U5, U6, U7, U8: Opamp_Dual, symbol Device:Opamp_Dual
- added C4: 10u, Capacitor_SMD:C_0603_1608Metric, symbol Device:C_Small
- added C45: 100n, Capacitor_SMD:C_0603_1608Metric, symbol Device:C
- added D13: led, LED_SMD:LED_0603_1608Metric, symbol Device:LED_Small
- added J4, J6: Conn_01x07, Connector_PinHeader_2.54mm:PinHeader_1x07_P2.54mm_Vertical, symbol Connector_Generic:Conn_01x07
- added R12: 10k, Resistor_SMD:R_0603_1608Metric, symbol Device:R
- added R5, R6: 27, Resistor_SMD:R_0603_1608Metric, symbol Device:R_Small
- added R56: 330, Resistor_SMD:R_0603_1608Metric, symbol Device:R
- added R8: 1k, Resistor_SMD:R_0603_1608Metric, symbol Device:R
- added SW3, SW4: SW_SPST, SamacSys_Parts:PTS526SK15SMTR2LFS, symbol Switch:SW_SPST
- added U16: M24C02-WMN, Package_SO:SOIC-8_3.9x4.9mm_P1.27mm, symbol Memory_EEPROM:M24C02-WMN
- added U3: MC74VHC4052DR2G, Package_SO:SOIC-16_3.9x9.9mm_P1.27mm, symbol My_custom_lib:MC74VHC4052DR2G
- C1, C10, C11, C15, C2, C3, C5, C6, C7, C8, C9: footprint Capacitor_SMD:C_0805_2012Metric_Pad1.18x1.45mm_HandSolder -> Capacitor_SMD:C_0603_1608Metric; LCSC (none) -> C14663
- C12: value 1u -> 100n; footprint Capacitor_SMD:C_0805_2012Metric_Pad1.18x1.45mm_HandSolder -> Capacitor_SMD:C_0603_1608Metric; LCSC (none) -> C14663
- D1: value LED_Small Red -> led; footprint LED_SMD:LED_0603_1608Metric_Pad1.05x0.95mm_HandSolder -> LED_SMD:LED_0603_1608Metric; LCSC (none) -> C72041
- FB1: footprint (none) -> Resistor_SMD:R_0603_1608Metric_Pad0.98x0.95mm_HandSolder
- J5: renamed from J1; now left out of the parts list
- R1: footprint Resistor_SMD:R_0603_1608Metric_Pad0.98x0.95mm_HandSolder -> Resistor_SMD:R_0603_1608Metric; LCSC (none) -> C23138
- R10, R17, R18, R19: footprint Resistor_SMD:R_0603_1608Metric_Pad0.98x0.95mm_HandSolder -> Resistor_SMD:R_0603_1608Metric; LCSC (none) -> C25804
- R11: renamed from R9; footprint Resistor_SMD:R_0603_1608Metric_Pad0.98x0.95mm_HandSolder -> Resistor_SMD:R_0603_1608Metric; LCSC (none) -> C23189
- R13, R16: value e -> 10k; footprint Resistor_SMD:R_0603_1608Metric_Pad0.98x0.95mm_HandSolder -> Resistor_SMD:R_0603_1608Metric; LCSC (none) -> C25804
- R14, R15: value 10Meg -> 10k; footprint Resistor_SMD:R_0603_1608Metric_Pad0.98x0.95mm_HandSolder -> Resistor_SMD:R_0603_1608Metric; LCSC (none) -> C25804
- R2, R4: footprint Resistor_SMD:R_0603_1608Metric_Pad0.98x0.95mm_HandSolder -> Resistor_SMD:R_0603_1608Metric; LCSC (none) -> C21190
- R20: value 10k -> 5k6; footprint Resistor_SMD:R_0603_1608Metric_Pad0.98x0.95mm_HandSolder -> Resistor_SMD:R_0603_1608Metric; LCSC (none) -> C23189
- R21: value 1k -> 5k6; footprint Resistor_SMD:R_0603_1608Metric_Pad0.98x0.95mm_HandSolder -> Resistor_SMD:R_0603_1608Metric; LCSC (none) -> C23189
- R3: now left out of the parts list
- R7: value 1k -> 220k; footprint Resistor_SMD:R_0603_1608Metric_Pad0.98x0.95mm_HandSolder -> Resistor_SMD:R_0603_1608Metric; LCSC (none) -> C22961
- R9: renamed from R8; footprint Resistor_SMD:R_0603_1608Metric_Pad0.98x0.95mm_HandSolder -> Resistor_SMD:R_0603_1608Metric; LCSC (none) -> C25804
- SW1: renamed from SW2; LCSC (none) -> C318884
- U2: LCSC (none) -> C97521
- U4: renamed from U3; LCSC (none) -> C2040
- renumbered J2 to J1, J3 to J2, SW1 to SW2, U4 to U5
Connections:
- net GPIO10 is gone; now on net I2C_SDA: U4.13 (GPIO10)
- net GPIO18 is gone; now on net FB2: U4.29 (GPIO18)
- net +3V3: now also R18.2, R19.2, R2.1, R20.2, R21.2, R7.2, SW2.11, SW2.12, SW2.13, C4.1, C45.1, J4.7 (Pin_7), J6.6 (Pin_6), R56.2, U16.1 (E0), U16.2 (E1), U16.3 (E2), U16.7 (~{WC}), U16.8 (VCC), U3.16 (VCC); no longer R2.2
- net D+: now also R5.2
- net D-: now also R6.2
- net GND: now also R11.1, R13.1, R16.1, SW2.7, C4.2, C45.2, D13.1 (K), J4.1 (Pin_1), J4.6 (Pin_6), J6.1 (Pin_1), J6.4 (Pin_4), R12.1, SW3.1 (A), SW4.1 (A), U16.4 (VSS), U3.8 (GND); no longer R10.1, R18.1, R19.1, R20.1
- net GPIO0: now also R17.2, SW2.1; no longer R20.2, SW2.2
- net GPIO1: now also R16.2, SW2.2; no longer R19.2, SW2.1
- net GPIO2: now also R15.2, SW2.3
- net GPIO23: now also R7.1, U3.6 (ENABLE)
- net GPIO24: now also U3.9 (B); no longer R10.2, R11.1
- net GPIO25: now also U3.10 (A)
- net GPIO28_ADC2: now also U3.3 (Y)
- net GPIO29_ADC3: now also U3.13 (X)
- net GPIO3: now also R14.2, SW2.4
- net GPIO4: now also R13.2, SW2.5
- net GPIO5: now also SW2.6, R12.2
- net RUN: now also SW2.10
- net USB+: now also R5.1
- net USB-: now also R6.1
- net VBUS: now also R10.2; no longer R11.2
- net XOUT: now also R8.1; no longer R7.1
- net XOUT-raw: now also R8.2; no longer R7.2
- net input: now also U3.1 (Y0); no longer R16.1, R18.2
- net output: now also U3.12 (X0); no longer R13.1, R17.2
- net V_ADC: now reaches C11.1, U1.1 (K), U4.43 (ADC_AVDD)
- net V_ADC: now also R2.2, J6.5 (Pin_5); no longer R2.1
- net +12V renamed I2C_SDA
- net I2C_SDA: now also J6.3 (Pin_3), U16.5 (SDA)
- net GPIO11 renamed I2C_SCL
- net I2C_SCL: now also R20.1, J6.2 (Pin_2), U16.6 (SCL)
- net GPIO12 renamed SPI_MISO
- net SPI_MISO: now also J4.3 (Pin_3)
- net GPIO13 renamed SPI_SS
- net SPI_SS: now also J4.5 (Pin_5)
- net GPIO14 renamed SPI_SCK
- net SPI_SCK: now also J4.2 (Pin_2)
- net GPIO15 renamed SPI_MOSI
- net SPI_MOSI: now also J4.4 (Pin_4)
- net GPIO16 renamed Button_down
- net Button_down: now also R18.1, SW3.2 (B)
- net GPIO17 renamed Button_up
- net Button_up: now also R19.1, SW4.2 (B)
- net GPIO8 renamed Buck_pwm1
- net GPIO9 renamed Buck_pwm2
- new net: D13.2 (A), R56.1
- new net -VDC: U3.7 (VEE)
- new net 1v1_buffered: J6.7 (Pin_7)
- new net USB_V: R10.1, R11.2, U3.15 (X2)
- new net current_LDO: U3.4 (Y3)
- new net current_in: U3.5 (Y1)
- new net current_out: U3.14 (X1)
- new net output_LDO: U3.11 (X3)
- no-connect marks 2 -> 3
Other:
- added sheet LDO (LDO.kicad_sch)
- added sheet MCU_POWER (MCU_POWER.kicad_sch)
- added sheet SMPS (SMPS.kicad_sch)
- note removed: "FB voltage set to 1.5V"
- note removed: "For ourput (1.5V FB): 1.8v 2k 2v 3.33k 3.3v 12k 5v 23.3k 12v 70k 24 150k 48 310k 0.2v FB: 1v 40k"
- note removed: "with 12V in 2A out: inductor/FET current 1v D= 8.8% Imax=22.5A 48A 3.3v Imax=7.27A 14.5A 5V Imax=4.8A 9.6A 48V D=76% Imax=0.5A 4.3A 120V Imax=0.2A 4.3A"
- moved on the sheet: D1, J5, R1, R11, SW2
