File: RP2040_SMPS/RP2040_SMPS.kicad_pcb (KiCad board)
At the start: 2 copper layers, 58 parts, among them J1 debug, J2 Conn_01x02, J3 USB_B_Mini, J4 Conn_01x01, J7 Conn_01x01, SW1 SW_SPST, SW2 SW_SPST, U1 LM4040DBZ-3.0, U2 W25Q128JVS, U3 RP2040, U4 D1213A-02SM, Y1 ABLS-12.000MHZ-B4-T

Commit message: j
Parts:
- removed FB1: HI1806T600R-10, SamacSys_Parts:BEADC4516X185N
- removed J3: USB_B_Mini, Connector_USB:USB_Mini-B_Lumberg_2486_01_Horizontal
- removed J7: Conn_01x01, Connector_PinSocket_2.54mm:PinSocket_1x01_P2.54mm_Vertical
- added C19: 10u@50V, Capacitor_SMD:C_0805_2012Metric_Pad1.18x1.45mm_HandSolder, F.Cu at (187.9, 117.6)
- added C20: 100n, Capacitor_SMD:C_0805_2012Metric_Pad1.18x1.45mm_HandSolder, F.Cu at (178.2, 117.6)
- added C21: 100n, Capacitor_SMD:C_0805_2012Metric_Pad1.18x1.45mm_HandSolder, F.Cu at (195.7, 114.0)
- added C22: 100n, Capacitor_SMD:C_0805_2012Metric_Pad1.18x1.45mm_HandSolder, F.Cu at (183.1, 117.6)
- added C23: 100n, Capacitor_SMD:C_0805_2012Metric_Pad1.18x1.45mm_HandSolder, F.Cu at (183.1, 120.6)
- added C24: 100n, Capacitor_SMD:C_0805_2012Metric_Pad1.18x1.45mm_HandSolder, F.Cu at (178.2, 120.6)
- added C25: 10u@50V, Capacitor_SMD:C_0805_2012Metric_Pad1.18x1.45mm_HandSolder, F.Cu at (269.2, 68.4)
- added C26: 10u@50V, Capacitor_SMD:C_0805_2012Metric_Pad1.18x1.45mm_HandSolder, F.Cu at (277.7, 62.1)
- added C27: 10u@50V, Capacitor_SMD:C_0805_2012Metric_Pad1.18x1.45mm_HandSolder, F.Cu at (284.0, 58.9)
- added C28: 10u@50V, Capacitor_SMD:C_0805_2012Metric_Pad1.18x1.45mm_HandSolder, F.Cu at (286.1, 54.1)
- added C29: 10u@50V, Capacitor_SMD:C_0805_2012Metric_Pad1.18x1.45mm_HandSolder, F.Cu at (271.3, 65.3)
- added C30: 10u@50V, Capacitor_SMD:C_0805_2012Metric_Pad1.18x1.45mm_HandSolder, F.Cu at (277.7, 65.1)
- added C35: 100n, Capacitor_SMD:C_0805_2012Metric_Pad1.18x1.45mm_HandSolder, F.Cu at (269.2, 71.4)
- added C36: 100n, Capacitor_SMD:C_0805_2012Metric_Pad1.18x1.45mm_HandSolder, F.Cu at (274.0, 68.3)
- added C37: 100n, Capacitor_SMD:C_0805_2012Metric_Pad1.18x1.45mm_HandSolder, F.Cu at (286.1, 51.1)
- added C38: 100n, Capacitor_SMD:C_0805_2012Metric_Pad1.18x1.45mm_HandSolder, F.Cu at (290.9, 51.1)
- added C39: 100n, Capacitor_SMD:C_0805_2012Metric_Pad1.18x1.45mm_HandSolder, F.Cu at (245.8, 104.7)
- added C40: 10u, Capacitor_SMD:C_0603_1608Metric_Pad1.08x0.95mm_HandSolder, F.Cu at (241.8, 107.8)
- added C41: 10u, Capacitor_SMD:C_0603_1608Metric_Pad1.08x0.95mm_HandSolder, F.Cu at (249.7, 99.5)
- added C42: 100n, Capacitor_SMD:C_0805_2012Metric_Pad1.18x1.45mm_HandSolder, F.Cu at (237.2, 108.0)
- added C43: 10u, Capacitor_SMD:C_0603_1608Metric_Pad1.08x0.95mm_HandSolder, F.Cu at (237.0, 113.3)
- added C44: 10u, Capacitor_SMD:C_0603_1608Metric_Pad1.08x0.95mm_HandSolder, F.Cu at (237.0, 110.8)
- added D10: SS210, Diode_SMD:D_SMA_Handsoldering, F.Cu at (232.6, 97.2)
- added D11: B5819W_SL, Diode_SMD:D_SOD-123, F.Cu at (230.5, 115.4)
- added D12: B5819W_SL, Diode_SMD:D_SOD-123, F.Cu at (250.4, 96.6)
- added D2: ZMM3V3-M, Diode_SMD:D_MiniMELF, F.Cu at (215.6, 96.5)
- added D3: 18v, Diode_THT:D_5KPW_P7.62mm_Vertical_AnodeUp, F.Cu at (258.9, 54.4)
- added D4: ZMM3V3-M, Diode_SMD:D_MiniMELF, F.Cu at (278.4, 59.0)
- added D7: ZMM3V3-M, Diode_SMD:D_MiniMELF, F.Cu at (257.3, 75.0)
- added D8: B5819W_SL, Diode_SMD:D_SOD-123, F.Cu at (240.5, 104.8)
- added D9: SS210, Diode_SMD:D_SMA_Handsoldering, F.Cu at (232.6, 101.7)
- added HS1: Heatsink_Pad_2Pin, Z_mycustom_footprint_lib:HSE-B20500-040H, F.Cu at (194.1, 102.2)
- added J10: Conn_01x01, Connector_PinSocket_2.54mm:PinSocket_1x01_P2.54mm_Vertical, F.Cu at (282.4, 62.9)
- added J11: jumper, Connector_PinHeader_2.54mm:PinHeader_2x03_P2.54mm_Vertical, F.Cu at (229.9, 106.3)
- added J5: debug, Connector_PinSocket_2.54mm:PinSocket_1x03_P2.54mm_Vertical, F.Cu at (209.5, 66.3)
- added J6: Conn_01x07, Connector_PinHeader_2.54mm:PinHeader_1x07_P2.54mm_Vertical, F.Cu at (194.2, 51.9)
- added Q1: Q_PMOS_DGS, Package_TO_SOT_THT:TO-247-3_Vertical, F.Cu at (179.1, 112.6)
- added Q3: HYG025N06LS1C2, Z_mycustom_footprint_lib:DFN-8_(5x6), F.Cu at (280.5, 50.8)
- added Q4: HYG025N06LS1C2, Z_mycustom_footprint_lib:DFN-8_(5x6), F.Cu at (263.6, 68.2)
- added Q5: HYG025N06LS1C2, Z_mycustom_footprint_lib:DFN-8_(5x6), F.Cu at (257.2, 66.8)
- added Q6: HYG025N06LS1C2, Z_mycustom_footprint_lib:DFN-8_(5x6), F.Cu at (265.7, 60.4)
- added Q7: HYG025N06LS1C2, Z_mycustom_footprint_lib:DFN-8_(5x6), F.Cu at (272.0, 57.3)
- added R11: 5k6, Resistor_SMD:R_0603_1608Metric, F.Cu at (246.8, 53.4)
- added R12: 10k, Resistor_SMD:R_0603_1608Metric, F.Cu at (213.6, 53.4)
- added R23: 220k, Resistor_SMD:R_0603_1608Metric, F.Cu at (219.2, 99.4)
- added R24: 100k, Resistor_SMD:R_0603_1608Metric, F.Cu at (187.5, 120.3)
- added R25: 1k, Resistor_SMD:R_0603_1608Metric, F.Cu at (195.3, 116.7)
- added R26: 10k, Resistor_SMD:R_0603_1608Metric, F.Cu at (195.5, 119.2)
- added R27: 10k, Resistor_SMD:R_0603_1608Metric, F.Cu at (214.4, 102.4)
- added R28: 10k, Resistor_SMD:R_0603_1608Metric, F.Cu at (220.8, 96.2)
- added R29: 10k, Resistor_SMD:R_0603_1608Metric, F.Cu at (204.9, 110.7)
- added R30: 100k, Resistor_SMD:R_0603_1608Metric, F.Cu at (191.5, 120.3)
- added R31: 100k, Resistor_SMD:R_0603_1608Metric, F.Cu at (204.9, 113.2)
- added R32: 1k, Resistor_SMD:R_0603_1608Metric, F.Cu at (214.4, 104.9)
- added R33: 1k, Resistor_SMD:R_0603_1608Metric, F.Cu at (199.3, 116.7)
- added R34: 1k, Resistor_SMD:R_0603_1608Metric, F.Cu at (200.1, 113.7)
- added R35: 1k, Resistor_SMD:R_0603_1608Metric, F.Cu at (199.5, 119.2)
- added R38: 1k, Resistor_SMD:R_0603_1608Metric, F.Cu at (268.8, 74.2)
- added R39: 220k, Resistor_SMD:R_0603_1608Metric, F.Cu at (262.5, 76.0)
- added R40: 220k, Resistor_SMD:R_0603_1608Metric, F.Cu at (294.5, 53.9)
- added R41: 10k, Resistor_SMD:R_0603_1608Metric, F.Cu at (272.8, 74.2)
- added R42: 10k, Resistor_SMD:R_0603_1608Metric, F.Cu at (295.3, 50.8)
- added R43: 27, Resistor_SMD:R_0603_1608Metric, F.Cu at (288.4, 59.4)
- added R44: 27, Resistor_SMD:R_0603_1608Metric, F.Cu at (278.4, 67.9)
- added R45: 27, Resistor_SMD:R_0603_1608Metric, F.Cu at (276.8, 73.6)
- added R46: 27, Resistor_SMD:R_0603_1608Metric, F.Cu at (290.5, 53.9)
- added R47: 1k, Resistor_SMD:R_0603_1608Metric, F.Cu at (277.6, 71.1)
- added R48: 1k, Resistor_SMD:R_0603_1608Metric, F.Cu at (288.4, 56.9)
- added R49: 1k, Resistor_SMD:R_0603_1608Metric, F.Cu at (292.4, 56.4)
- added R50: 1k, Resistor_SMD:R_0603_1608Metric, F.Cu at (273.6, 71.1)
- added R51: 1k, Resistor_SMD:R_0603_1608Metric, F.Cu at (241.2, 113.3)
- added R52: 100k, Resistor_SMD:R_0603_1608Metric, F.Cu at (246.0, 107.4)
- added R53: 100k, Resistor_SMD:R_0603_1608Metric, F.Cu at (241.2, 110.8)
- added R54: 10k, Resistor_SMD:R_0603_1608Metric, F.Cu at (235.3, 115.8)
- added R55: 10k, Resistor_SMD:R_0603_1608Metric, F.Cu at (250.2, 102.0)
- added SW3: SW_SPST, SamacSys_Parts:PTS526SK15SMTR2LFS, F.Cu at (221.2, 53.7)
- added SW4: SW_SPST, SamacSys_Parts:PTS526SK15SMTR2LFS, F.Cu at (210.6, 59.8)
- added U10: LM5109BMA, Package_SO:SOIC-8_3.9x4.9mm_P1.27mm, F.Cu at (273.1, 52.8)
- added U13: AMS1117-3.3, Package_TO_SOT_SMD:SOT-223-3_TabPin2, F.Cu at (242.6, 99.0)
- added U5: D1213A-02SM, Package_TO_SOT_SMD:SOT-23-5_HandSoldering, F.Cu at (237.1, 51.9)
- added U9: LM5109BMA, Package_SO:SOIC-8_3.9x4.9mm_P1.27mm, F.Cu at (258.3, 62.4)
- C12: value 1u -> 100n
- C16: value y -> 10u@50V
- C17: value x -> 10u@50V
- C18: value z -> 10u@50V
- C4: value 22u -> 100n
- J1: value debug -> Conn_01x02; footprint Connector_PinSocket_2.54mm:PinSocket_1x03_P2.54mm_Vertical -> Connector_PinHeader_2.54mm:PinHeader_1x02_P2.54mm_Vertical
- J2: value Conn_01x02 -> USB_B_Mini; footprint Connector_PinHeader_2.54mm:PinHeader_1x02_P2.54mm_Vertical -> Connector_USB:USB_A_Molex_67643_Horizontal
- J4: value Conn_01x01 -> Conn_01x07; footprint Connector_PinSocket_2.54mm:PinSocket_1x01_P2.54mm_Vertical -> Connector_PinHeader_2.54mm:PinHeader_1x07_P2.54mm_Vertical
- R10, R17, R18, R19, R2, R4, R5, R6: footprint Resistor_SMD:R_0603_1608Metric_Pad0.98x0.95mm_HandSolder -> Resistor_SMD:R_0603_1608Metric
- R13, R16: value e -> 10k; footprint Resistor_SMD:R_0603_1608Metric_Pad0.98x0.95mm_HandSolder -> Resistor_SMD:R_0603_1608Metric
- R14, R15: value 10Meg -> 10k; footprint Resistor_SMD:R_0603_1608Metric_Pad0.98x0.95mm_HandSolder -> Resistor_SMD:R_0603_1608Metric
- R20: value 10k -> 5k6; footprint Resistor_SMD:R_0603_1608Metric_Pad0.98x0.95mm_HandSolder -> Resistor_SMD:R_0603_1608Metric
- R21: value 1k -> 5k6; footprint Resistor_SMD:R_0603_1608Metric_Pad0.98x0.95mm_HandSolder -> Resistor_SMD:R_0603_1608Metric
- R7: value 1k -> 220k; footprint Resistor_SMD:R_0603_1608Metric_Pad0.98x0.95mm_HandSolder -> Resistor_SMD:R_0603_1608Metric
- R8: value 10k -> 1k; footprint Resistor_SMD:R_0603_1608Metric_Pad0.98x0.95mm_HandSolder -> Resistor_SMD:R_0603_1608Metric
- R9: value 5k6 -> 10k; footprint Resistor_SMD:R_0603_1608Metric_Pad0.98x0.95mm_HandSolder -> Resistor_SMD:R_0603_1608Metric
- SW2: value SW_SPST -> SW_DIP_x08; footprint SamacSys_Parts:PTS526SK15SMTR2LFS -> Button_Switch_THT:SW_DIP_SPSTx08_Slide_9.78x22.5mm_W7.62mm_P2.54mm
- U3: value RP2040 -> MC74VHC4052DR2G; footprint RP2040_minimal:RP2040-QFN-56 -> Package_SO:SOIC-16_3.9x9.9mm_P1.27mm
- U4: value D1213A-02SM -> RP2040; footprint Package_TO_SOT_SMD:SOT-23-5_HandSoldering -> RP2040_minimal:RP2040-QFN-56
- moved H1 196.6 mm to (55.0, 145.0)
- moved H4 171.9 mm to (55.0, 55.0)
- moved H2 84.3 mm to (145.0, 145.0)
- moved H3 70.8 mm to (145.0, 55.0)
- moved R13 62.5 mm to (240.4, 61.5)
- moved C18 61.5 mm to (200.5, 111.0)
- moved J4 56.7 mm to (189.6, 51.9)
- moved C16 46.8 mm to (214.8, 99.7)
- moved R3 46.8 mm to (242.1, 53.9)
- moved SW2 46.1 mm to (177.8, 52.8)
- moved R8 45.4 mm to (213.6, 50.8)
- moved R10 38.3 mm to (241.2, 58.9)
- moved J1 37.2 mm to (227.2, 60.2)
- moved R7 37.0 mm to (231.7, 67.3)
- moved C2 35.8 mm to (242.4, 51.1)
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Connections:
- net /GPIO11 renamed /current_out
- net /GPIO8 renamed /output_LDO
- C11 pad 1: Net-(C11-Pad1) -> /V_ADC
- C16 pad 1: Net-(C16-Pad1) -> Net-(Q1-Pad3)
- C17 pad 1: Net-(C17-Pad1) -> Net-(Q1-Pad3)
- C18 pad 1: Net-(C18-Pad1) -> Net-(J7-Pad2)
- J1 pad 1: /SWCLK -> /~{USB_BOOT}
- J2 pad 1: /~{USB_BOOT} -> /VBUS_RAW
- J2 pad 2: GND -> D-
- J4 pad 1: Net-(J3-Pad6) -> GND
- R10 pad 1: GND -> /USB_V
- R10 pad 2: GPIO24 -> VBUS
- R13 pad 1: /output -> GND
- R13 pad 2: Net-(C18-Pad1) -> /GPIO4
- R14 pad 2: Net-(C18-Pad1) -> /GPIO3
- R15 pad 2: Net-(C16-Pad1) -> /GPIO2
- R16 pad 1: /input -> GND
- R16 pad 2: Net-(C16-Pad1) -> /GPIO1
- R17 pad 2: /output -> /GPIO0
- R18 pad 1: GND -> /Button_down
- R18 pad 2: /input -> +3V3
- R19 pad 1: GND -> /Button_up
- R19 pad 2: /GPIO0 -> +3V3
- R2 pad 1: Net-(C11-Pad1) -> +3V3
- R2 pad 2: +3V3 -> /V_ADC
- R20 pad 1: GND -> I2C_SCL
- R20 pad 2: /GPIO1 -> +3V3
- R21 pad 1: Net-(J6-Pad2) -> I2C_SDA
- R21 pad 2: Net-(Q5-Pad2) -> +3V3
- R5 pad 1: D+ -> /USB+
- R5 pad 2: /USB+ -> D+
- R6 pad 1: D- -> /USB-
- R6 pad 2: /USB- -> D-
- R7 pad 1: /XOUT -> /GPIO23
- R7 pad 2: /XOUT-raw -> +3V3
- R8 pad 1: /RUN -> /XOUT
- R8 pad 2: +3V3 -> /XOUT-raw
- R9 pad 1: GPIO24 -> /RUN
- R9 pad 2: VBUS -> +3V3
- SW1 pad 2: /~{USB_BOOT} -> /RUN
- SW2 pad 1: GND -> /GPIO0
- SW2 pad 2: /RUN -> /GPIO1
- U1 pad 1: Net-(C11-Pad1) -> /V_ADC
- U3 pad 1: +3V3 -> /input
- U3 pad 10: +3V3 -> /GPIO25
- U3 pad 12: /GPIO9 -> /output
- U3 pad 13: /GPIO10 -> /GPIO29_ADC3
- U3 pad 15: /GPIO12 -> /USB_V
- U3 pad 16: /GPIO13 -> +3V3
- U3 pad 2: /GPIO0 -> unconnected-(U3-Pad2)
- U3 pad 3: /GPIO1 -> /GPIO28_ADC2
- U3 pad 4: /GPIO2 -> /current_LDO
- U3 pad 5: /GPIO3 -> /current_in
- U3 pad 6: /GPIO4 -> /GPIO23
- U3 pad 7: /GPIO5 -> -VDC
- U3 pad 8: /GPIO6 -> GND
- U3 pad 9: /GPIO7 -> /GPIO24
- U4 pad 1: unconnected-(U4-Pad1) -> +3V3
- U4 pad 2: GND -> /GPIO0
- U4 pad 3: D- -> /GPIO1
- U4 pad 4: D+ -> /GPIO2
- U4 pad 5: VBUS -> /GPIO3
Other:
- board outline added: 100 x 100 mm
